File: tfm_pcb.kicad_sch (KiCad schematic)
At the start: 74 parts, among them J1 Conn_01x02_MountingPin, J11 Conn_01x01_Pin, J12 Conn_01x01_Pin, J13 Conn_01x01_Pin, J14 Conn_01x01_Pin, J15 Conn_01x01_Socket, J16 Conn_01x01_Socket, J17 Conn_01x01_Socket, J18 Conn_01x01_Socket, J19 Conn_01x01_Socket, J2 USB_B_Micro, J20 Conn_01x01_Socket, J21 Conn_01x01_Socket, J22 Conn_01x01_Socket, J23 Conn_01x01_Socket, J24 Conn_01x01_Socket, J3 Mounting Pin, J4 Conn_01x01_Pin, J5 Conn_01x01_Pin, J6 Conn_01x01_Pin, U1 ESP32-S3-WROOM-2, U2 MCP73871-2CC, U3 ADS1292IPBS, U4 LSM6DS3, U5 USBLC6-2SC6, U6 XC6220B331MR, U7 USBLC6-2SC6

Commit message: Cambios envío a Roberto 06-09
Parts:
- removed J11: Conn_01x01_Pin, TestPoint:TestPoint_Pad_D1.0mm, symbol Connector:Conn_01x01_Pin

Commit message: cambios
Parts:
- removed J14, J4: Conn_01x01_Pin, TestPoint:TestPoint_Pad_D1.0mm, symbol Connector:Conn_01x01_Pin
- removed R15: 0, Resistor_SMD:R_0603_1608Metric, symbol Device:R
- C12: value 1u -> 10u
- FB1: footprint Resistor_SMD:R_0603_1608Metric -> Inductor_SMD:L_0603_1608Metric
Connections:
- net GNDA is gone; now on net GND: C10.2, C11.2, C12.1, C13.1, C6.1, C7.1, C8.2, C9.1, J13.1 (Pin_1), J20.1 (Pin_1), J21.1 (Pin_1), J22.1 (Pin_1), J23.1 (Pin_1), J24.1 (Pin_1), U3.10 (VREFN), U3.13 (AVSS), U3.16 (START), U3.24 (DGND)
- net +3.3V: now also FB1.1; no longer FB1.2
- net +3.3VA: now also FB1.2; no longer FB1.1
