File: tfm_pcb.kicad_sch (KiCad schematic)
At the start: 67 parts, among them J1 Conn_01x02_MountingPin, J12 Conn_01x01_Pin, J13 Conn_01x01_Pin, J2 USB_B_Micro, J3 Mounting Pin, J4 Conn_01x10_Pin, J5 Conn_01x01_Pin, J6 Conn_01x01_Pin, U1 ESP32-S3-WROOM-2, U2 MCP73871-2CC, U3 ADS1292IPBS, U4 LSM6DS3, U5 USBLC6-2SC6, U6 XC6220B331MR, U7 USBLC6-2SC6

Commit message: Añadimos USB tipo C y mejoras en el ruteo
Parts:
- removed J2: USB_B_Micro, Connector_USB:USB_Micro-B_Molex-105017-0001, symbol Connector:USB_B_Micro
- added J7: USB_C_Receptacle_USB2.0_16P, Connector_USB:USB_C_Receptacle_HCTL_HC-TYPE-C-16P-01A, symbol Connector:USB_C_Receptacle_USB2.0_16P
- added R20, R21: 5.1k, Resistor_SMD:R_0603_1608Metric, symbol Device:R
- C12: footprint Capacitor_SMD:C_0402_1005Metric -> Capacitor_SMD:C_0603_1608Metric
Connections:
- net +5V: now also J7.A4 (VBUS), J7.A9 (VBUS), J7.B4 (VBUS), J7.B9 (VBUS)
- net GND: now also J7.A1 (GND), J7.A12 (GND), J7.B1 (GND), J7.B12 (GND), J7.SH (SHIELD), R20.2, R21.2
- net at U5.1 (I/O1): now also J7.A7 (D-), J7.B7 (D-)
- net at U5.3 (I/O2): now also J7.A6 (D+), J7.B6 (D+)
- net VSYS: now reaches C22.1, C4.1, U2.1 (OUT), U2.20 (OUT), U6.1 (VIN), U6.3 (CE)
- new net: J7.A5 (CC1), R21.1
- new net: J7.B5 (CC2), R20.1
- no-connect marks 20 -> 21
Other:
- moved on the sheet: U5
