File: tfm_pcb.kicad_pcb (KiCad board)
At the start: 2 copper layers, 73 x 55 mm, 67 parts, among them J1 Conn_01x02_MountingPin, J12 Conn_01x01_Pin, J13 Conn_01x01_Pin, J2 USB_B_Micro, J3 Mounting Pin, J4 Conn_01x10_Pin, J5 Conn_01x01_Pin, J6 Conn_01x01_Pin, U1 ESP32-S3-WROOM-2, U2 MCP73871-2CC, U3 ADS1292IPBS, U4 LSM6DS3, U5 USBLC6-2SC6, U6 XC6220B331MR, U7 USBLC6-2SC6

Commit message: Condensadores del ADS1292 en 0402 (C8, C11, C12, C13) y recolocación de VREF
- Esquemático y PCB sincronizados: C8, C11, C12 y C13 en 0402.
- C12/C13 (VREFP) más cerca del pin 9; punto de prueba de VREF recolocado.
- Retoques de rutado del autor en VREF, GND, +3.3V, +3.3VA, RX y EN.

Pendiente: el punto de prueba J12 aparece como "VREF" solo en la PCB
(paridad); alivios térmicos de C11.2 y U4.7; dos pistas colgando.

Co-Authored-By: Claude Opus 5.5 <noreply@anthropic.com>
Parts:
- C12, C13: footprint Capacitor_SMD:C_0603_1608Metric -> Capacitor_SMD:C_0402_1005Metric
- moved C12 2.02 mm to (162.3, 89.0)
- moved VREF 1.76 mm to (164.6, 89.5)
- moved C13 1.36 mm to (161.2, 89.0)
- renumbered J12 to VREF
Routing:
- net +3.3V: track 169.4 -> 191.2 mm
- net /VREF: track 8.14 -> 5.95 mm
- net GND: track 16.3 -> 18.3 mm, vias 108 -> 109
