File: tfm_pcb.kicad_pcb (KiCad board)
At the start: 2 copper layers, 73 x 55 mm, 67 parts, among them J1 Conn_01x02_MountingPin, J13 Conn_01x01_Pin, J2 USB_B_Micro, J3 Mounting Pin, J4 Conn_01x10_Pin, J5 Conn_01x01_Pin, J6 Conn_01x01_Pin, U1 ESP32-S3-WROOM-2, U2 MCP73871-2CC, U3 ADS1292IPBS, U4 LSM6DS3, U5 USBLC6-2SC6, U6 XC6220B331MR, U7 USBLC6-2SC6

Commit message: Añadimos USB tipo C y mejoras en el ruteo
Parts:
- removed J2: USB_B_Micro, Connector_USB:USB_Micro-B_Molex-105017-0001
- added J7: USB_C_Receptacle_USB2.0_16P, Connector_USB:USB_C_Receptacle_HCTL_HC-TYPE-C-16P-01A, F.Cu at (108.0, 72.9)
- added R20: 5.1k, Resistor_SMD:R_0603_1608Metric, F.Cu at (116.0, 76.5)
- added R21: 5.1k, Resistor_SMD:R_0603_1608Metric, F.Cu at (116.0, 70.3)
- C12: footprint Capacitor_SMD:C_0402_1005Metric -> Capacitor_SMD:C_0603_1608Metric
- moved J12 2.14 mm to (165.0, 91.6)
- moved C12 1.68 mm to (163.9, 89.5), turned to 180 degrees
- renumbered VREF to J12
Connections:
- net Net-(U6-CE) renamed /VSYS
Routing:
- net +3.3VA: track 23.1 -> 31.8 mm, vias 0 -> 2
- net Net-(J7-CC2): track 0.00 -> 4.26 mm
- net Net-(J7-CC1): track 0.00 -> 4.02 mm
- net /SHIELD: track 39.6 -> 42.8 mm
- net /VREF: track 5.95 -> 8.04 mm
- net +5V: track 95.6 -> 97.4 mm
- net +3.3V: track 191.2 -> 192.2 mm
- net GND: track 18.3 -> 19.3 mm, vias 109 -> 112
- net /EL2P: track 7.71 -> 8.37 mm
